File: magnetic_encoder.kicad_pcb (KiCad board)
At the start: 4 copper layers, 30 x 30 mm, 10 parts, among them J1 Conn_01x03_Pin, J2 Conn_01x04_Pin, J3 Conn_01x06_Pin, J4 Conn_01x01_Pin, U1 MT6835GT_STD

Commit message: added labels to pins
Connections:
- net CSK  renamed CSEL
Other:
- board text added: "5V"
- board text added: "A B Z PWM"
- board text added: "CPIO"
- board text added: "CS"
- board text added: "GND"
- board text added: "PICO"
- board text added: "SCK"
- board text added: "U V W"
Changed lines of the file:
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@@
 	(net 2 "CIPO")
 	(net 3 "PWM_OUT")
-	(net 4 "CSK ")
+	(net 4 "CSEL")
 	(net 5 "Z_OUT")
 	(net 6 "CAL_EN")
@@
 			(layers "F.Cu" "F.Mask" "F.Paste")
 			(roundrect_rratio 0.25)
-			(net 4 "CSK ")
+			(net 4 "CSEL")
 			(pinfunction "CSN")
 			(pintype "input")
@@
 		(tags "connector JST PH horizontal")
 		(property "Reference" "J1"
-			(at 0 5.8 90)
+			(at -6.375 -2.275 0)
 			(layer "B.SilkS")
 			(effects
@@
 		(tags "connector JST PH horizontal")
 		(property "Reference" "J3"
-			(at 0 5.8 0)
+			(at 9.15 -1.5 270)
 			(layer "B.SilkS")
 			(effects
@@
 			(layers "B.Cu" "B.Mask" "B.Paste")
 			(roundrect_rratio 0.25)
-			(net 4 "CSK ")
+			(net 4 "CSEL")
 			(pinfunction "Pin_6")
 			(pintype "passive")
@@
 		(tags "connector JST PH horizontal")
 		(property "Reference" "J2"
-			(at 0 5.8 90)
+			(at 7.525 -2.825 0)
 			(layer "B.SilkS")
 			(effects
@@
 		)
 	)
+	(gr_text "U\nV\nW"
+		(at 146.875 104.025 0)
+		(layer "B.SilkS")
+		(effects
+			(font
+				(size 1 1)
+				(thickness 0.1)
+			)
+			(justify left bottom mirror)
+		)
+	)
+	(gr_text "A\nB\nZ\nPWM"
+		(at 154.25 105.2 0)
+		(layer "B.SilkS")
+		(effects
+			(font
+				(size 1 1)
+				(thickness 0.1)
+			)
+			(justify left bottom mirror)
+		)
+	)
+	(gr_text "CAL_EN"
+		(at 150.55 111.825 0)
+		(layer "B.SilkS")
+		(effects
+			(font
+				(size 1 1)
+				(thickness 0.1)
+			)
+			(justify left bottom mirror)
+		)
+	)
+	(gr_text "PICO"
+		(at 152.4 95.575 90)
+		(layer "B.SilkS")
+		(effects
+			(font
+				(size 1 1)
+				(thickness 0.1)
+			)
+			(justify left bottom mirror)
+		)
+	)
+	(gr_text "GND"
+		(at 148.325 95.625 90)
+		(layer "B.SilkS")
+		(effects
+			(font
+				(size 1 1)
+				(thickness 0.1)
+			)
+			(justify left bottom mirror)
+		)
+	)
+	(gr_text "CS"
+		(at 156.05 95.625 90)
+		(layer "B.SilkS")
+		(effects
+			(font
+				(size 1 1)
+				(thickness 0.1)
+			)
+			(justify left bottom mirror)
+		)
+	)
+	(gr_text "5V"
+		(at 146.275 95.725 90)
+		(layer "B.SilkS")
+		(effects
+			(font
+				(size 1 1)
+				(thickness 0.1)
+			)
+			(justify left bottom mirror)
+		)
+	)
+	(gr_text "SCK"
+		(at 154.425 95.4 90)
+		(layer "B.SilkS")
+		(effects
+			(font
+				(size 1 1)
+				(thickness 0.1)
+			)
+			(justify left bottom mirror)
+		)
+	)
+	(gr_text "CPIO"
+		(at 150.4 95.575 90)
+		(layer "B.SilkS")
+		(effects
+			(font
+				(size 1 1)
+				(thickness 0.1)
+			)
+			(justify left bottom mirror)
+		)
+	)
 	(segment
 		(start 152.8625 98.375)
@@
 		(polygon
 			(pts
-				(xy 135.425 114.7) (xy 164.675 114.725) (xy 164.675 85.55) (xy 135.425 85.55) (xy 135.425 85.55)
+				(xy 135.425 114.7) (xy 164.675 114.725) (xy 164.675 85.55) (xy 135.425 85.55)
 			)
 		)
